Commit message: Implemented ZMP, COM based standing domain

File: resources/robots/g1/urdf/g1_full_footpoint.urdf (robot description, URDF)
Before this commit: robot g1, 48 links, 47 joints
Links:
- removed link left_foot_1_link
- removed link left_foot_2_link
- removed link left_foot_3_link
- removed link left_foot_4_link
- added link left_footpoint_1_link, mass 0.001; collision sphere radius=0.001
- added link left_footpoint_2_link, mass 0.001; collision sphere radius=0.001
- added link left_footpoint_3_link, mass 0.001; collision sphere radius=0.001
- added link left_footpoint_4_link, mass 0.001; collision sphere radius=0.001
- added link left_footpoint_5_link, mass 0.001; collision sphere radius=0.001
- added link left_footpoint_6_link, mass 0.001; collision sphere radius=0.001
- added link right_footpoint_1_link, mass 0.001; collision sphere radius=0.001
- added link right_footpoint_2_link, mass 0.001; collision sphere radius=0.001
- added link right_footpoint_3_link, mass 0.001; collision sphere radius=0.001
- added link right_footpoint_4_link, mass 0.001; collision sphere radius=0.001
- added link right_footpoint_5_link, mass 0.001; collision sphere radius=0.001
- added link right_footpoint_6_link, mass 0.001; collision sphere radius=0.001
Joints:
- removed joint left_foot_1_joint
- removed joint left_foot_2_joint
- removed joint left_foot_3_joint
- removed joint left_foot_4_joint
- added joint left_footpoint_1_joint: type fixed, parent left_ankle_roll_link, child left_footpoint_1_link, origin xyz=0.12 0.025 -0.034 rpy=0 0 0
- added joint left_footpoint_2_joint: type fixed, parent left_ankle_roll_link, child left_footpoint_2_link, origin xyz=0.12 -0.025 -0.034 rpy=0 0 0
- added joint left_footpoint_3_joint: type fixed, parent left_ankle_roll_link, child left_footpoint_3_link, origin xyz=-0.045 0.025 -0.034 rpy=0 0 0
- added joint left_footpoint_4_joint: type fixed, parent left_ankle_roll_link, child left_footpoint_4_link, origin xyz=-0.045 -0.025 -0.034 rpy=0 0 0
- added joint left_footpoint_5_joint: type fixed, parent left_ankle_roll_link, child left_footpoint_5_link, origin xyz=-0.064 0 -0.034 rpy=0 0 0
- added joint left_footpoint_6_joint: type fixed, parent left_ankle_roll_link, child left_footpoint_6_link, origin xyz=0.138 0 -0.034 rpy=0 0 0
- added joint right_footpoint_1_joint: type fixed, parent right_ankle_roll_link, child right_footpoint_1_link, origin xyz=0.12 0.025 -0.034 rpy=0 0 0
- added joint right_footpoint_2_joint: type fixed, parent right_ankle_roll_link, child right_footpoint_2_link, origin xyz=0.12 -0.025 -0.034 rpy=0 0 0
- added joint right_footpoint_3_joint: type fixed, parent right_ankle_roll_link, child right_footpoint_3_link, origin xyz=-0.045 0.025 -0.034 rpy=0 0 0
- added joint right_footpoint_4_joint: type fixed, parent right_ankle_roll_link, child right_footpoint_4_link, origin xyz=-0.045 -0.025 -0.034 rpy=0 0 0
- added joint right_footpoint_5_joint: type fixed, parent right_ankle_roll_link, child right_footpoint_5_link, origin xyz=-0.064 0 -0.034 rpy=0 0 0
- added joint right_footpoint_6_joint: type fixed, parent right_ankle_roll_link, child right_footpoint_6_link, origin xyz=0.138 0 -0.034 rpy=0 0 0
