Commit message: Implemented footpoint-based training pipeline

File: resources/robots/g1/urdf/g1_full.urdf (robot description, URDF)
Before this commit: robot g1, 44 links, 43 joints
Links:
- added link left_footpoint_1_link, mass 0.010; collision sphere radius=0.001
- added link left_footpoint_2_link, mass 0.010; collision sphere radius=0.001
- added link left_footpoint_3_link, mass 0.010; collision sphere radius=0.001
- added link left_footpoint_4_link, mass 0.010; collision sphere radius=0.001
- added link left_footpoint_5_link, mass 0.010; collision sphere radius=0.001
- added link left_footpoint_6_link, mass 0.010; collision sphere radius=0.001
- added link right_footpoint_1_link, mass 0.010; collision sphere radius=0.001
- added link right_footpoint_2_link, mass 0.010; collision sphere radius=0.001
- added link right_footpoint_3_link, mass 0.010; collision sphere radius=0.001
- added link right_footpoint_4_link, mass 0.010; collision sphere radius=0.001
- added link right_footpoint_5_link, mass 0.010; collision sphere radius=0.001
- added link right_footpoint_6_link, mass 0.010; collision sphere radius=0.001
- link left_ankle_roll_link: geometry visual mesh filename=../meshes/left_ankle_roll_link.STL
- link right_ankle_roll_link: geometry visual mesh filename=../meshes/right_ankle_roll_link.STL
Joints:
- added joint left_footpoint_1_joint: type fixed, parent left_ankle_roll_link, child left_footpoint_1_link, origin xyz=0.12 0.025 -0.034 rpy=0 0 0
- added joint left_footpoint_2_joint: type fixed, parent left_ankle_roll_link, child left_footpoint_2_link, origin xyz=0.12 -0.025 -0.034 rpy=0 0 0
- added joint left_footpoint_3_joint: type fixed, parent left_ankle_roll_link, child left_footpoint_3_link, origin xyz=-0.045 0.025 -0.034 rpy=0 0 0
- added joint left_footpoint_4_joint: type fixed, parent left_ankle_roll_link, child left_footpoint_4_link, origin xyz=-0.045 -0.025 -0.034 rpy=0 0 0
- added joint left_footpoint_5_joint: type fixed, parent left_ankle_roll_link, child left_footpoint_5_link, origin xyz=-0.064 0 -0.034 rpy=0 0 0
- added joint left_footpoint_6_joint: type fixed, parent left_ankle_roll_link, child left_footpoint_6_link, origin xyz=0.138 0 -0.034 rpy=0 0 0
- added joint right_footpoint_1_joint: type fixed, parent right_ankle_roll_link, child right_footpoint_1_link, origin xyz=0.12 0.025 -0.034 rpy=0 0 0
- added joint right_footpoint_2_joint: type fixed, parent right_ankle_roll_link, child right_footpoint_2_link, origin xyz=0.12 -0.025 -0.034 rpy=0 0 0
- added joint right_footpoint_3_joint: type fixed, parent right_ankle_roll_link, child right_footpoint_3_link, origin xyz=-0.045 0.025 -0.034 rpy=0 0 0
- added joint right_footpoint_4_joint: type fixed, parent right_ankle_roll_link, child right_footpoint_4_link, origin xyz=-0.045 -0.025 -0.034 rpy=0 0 0
- added joint right_footpoint_5_joint: type fixed, parent right_ankle_roll_link, child right_footpoint_5_link, origin xyz=-0.064 0 -0.034 rpy=0 0 0
- added joint right_footpoint_6_joint: type fixed, parent right_ankle_roll_link, child right_footpoint_6_link, origin xyz=0.138 0 -0.034 rpy=0 0 0
