Commit message: debg

File: resources/robots/g1_description/g1_29dof_rev_1_0_ver3.urdf (robot description, URDF)
Before this commit: robot g1_29dof_rev_1_0, 40 links, 39 joints
Links:
- link head_link: geometry collision mesh filename=file:///root/unitree_rl_gym/resources/robots/g1_description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; visual mesh filename=file:///root/unitree_rl_gym/resources/robots/g1_description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
- link left_ankle_pitch_link: geometry collision mesh filename=file:///root/unitree_rl_gym/resources/robots/g1_description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; visual mesh filename=file:///root/unitree_rl_gym/resources/robots/g1_description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
- link left_ankle_roll_link: geometry collision box size=0.20820672 0.07558269 0.02; visual mesh filename=file:///root/unitree_rl_gym/resources/robots/g1_description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
- link left_elbow_link: geometry collision mesh filename=file:///root/unitree_rl_gym/resources/robots/g1_description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; visual mesh filename=file:///root/unitree_rl_gym/resources/robots/g1_description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
- link left_hip_pitch_link: geometry collision mesh filename=file:///root/unitree_rl_gym/resources/robots/g1_description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; visual mesh filename=file:///root/unitree_rl_gym/resources/robots/g1_description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
- link left_hip_roll_link: geometry collision mesh filename=file:///root/unitree_rl_gym/resources/robots/g1_description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; visual mesh filename=file:///root/unitree_rl_gym/resources/robots/g1_description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
- link left_hip_yaw_link: geometry collision mesh filename=file:///root/unitree_rl_gym/resources/robots/g1_description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; visual mesh filename=file:///root/unitree_rl_gym/resources/robots/g1_description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
- link left_knee_link: geometry collision mesh filename=file:///root/unitree_rl_gym/resources/robots/g1_description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; visual mesh filename=file:///root/unitree_rl_gym/resources/robots/g1_description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
- link left_shoulder_pitch_link: geometry collision cylinder length=0.05 radius=0.03; visual mesh filename=file:///root/unitree_rl_gym/resources/robots/g1_description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
- link left_shoulder_roll_link: geometry collision cylinder length=0.03 radius=0.03; visual mesh filename=file:///root/unitree_rl_gym/resources/robots/g1_description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
- link left_shoulder_yaw_link: geometry collision mesh filename=file:///root/unitree_rl_gym/resources/robots/g1_description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; visual mesh filename=file:///root/unitree_rl_gym/resources/robots/g1_description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
- link left_wrist_pitch_link: geometry collision mesh filename=file:///root/unitree_rl_gym/resources/robots/g1_description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; visual mesh filename=file:///root/unitree_rl_gym/resources/robots/g1_description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
- link left_wrist_roll_link: geometry collision mesh filename=file:///root/unitree_rl_gym/resources/robots/g1_description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; visual mesh filename=file:///root/unitree_rl_gym/resources/robots/g1_description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
- link left_wrist_yaw_link: geometry collision mesh filename=file:///root/unitree_rl_gym/resources/robots/g1_description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; visual mesh filename=file:///root/unitree_rl_gym/resources/robots/g1_description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
- link logo_link: geometry collision mesh filename=file:///root/unitree_rl_gym/resources/robots/g1_description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; visual mesh filename=file:///root/unitree_rl_gym/resources/robots/g1_description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
- link pelvis: geometry visual mesh filename=file:///root/unitree_rl_gym/resources/robots/g1_description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
- link pelvis_contour_link: geometry collision mesh filename=file:///root/unitree_rl_gym/resources/robots/g1_description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; visual mesh filename=file:///root/unitree_rl_gym/resources/robots/g1_description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
- link right_ankle_pitch_link: geometry collision mesh filename=file:///root/unitree_rl_gym/resources/robots/g1_description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; visual mesh filename=file:///root/unitree_rl_gym/resources/robots/g1_description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
- link right_ankle_roll_link: geometry collision box size=0.20820672 0.07558269 0.02; visual mesh filename=file:///root/unitree_rl_gym/resources/robots/g1_description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
- link right_elbow_link: geometry collision mesh filename=file:///root/unitree_rl_gym/resources/robots/g1_description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; visual mesh filename=file:///root/unitree_rl_gym/resources/robots/g1_description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
- link right_hip_pitch_link: geometry collision mesh filename=file:///root/unitree_rl_gym/resources/robots/g1_description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; visual mesh filename=file:///root/unitree_rl_gym/resources/robots/g1_description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
- link right_hip_roll_link: geometry collision mesh filename=file:///root/unitree_rl_gym/resources/robots/g1_description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; visual mesh filename=file:///root/unitree_rl_gym/resources/robots/g1_description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
- link right_hip_yaw_link: geometry collision mesh filename=file:///root/unitree_rl_gym/resources/robots/g1_description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; visual mesh filename=file:///root/unitree_rl_gym/resources/robots/g1_description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
- link right_knee_link: geometry collision mesh filename=file:///root/unitree_rl_gym/resources/robots/g1_description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; visual mesh filename=file:///root/unitree_rl_gym/resources/robots/g1_description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
- link right_rubber_hand: geometry collision box size=0.12 0.03 0.08; visual mesh filename=file:///root/unitree_rl_gym/resources/robots/g1_description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
- link right_shoulder_pitch_link: geometry collision cylinder length=0.05 radius=0.03; visual mesh filename=file:///root/unitree_rl_gym/resources/robots/g1_description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
- link right_shoulder_roll_link: geometry collision cylinder length=0.03 radius=0.03; visual mesh filename=file:///root/unitree_rl_gym/resources/robots/g1_description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
- link right_shoulder_yaw_link: geometry collision mesh filename=file:///root/unitree_rl_gym/resources/robots/g1_description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; visual mesh filename=file:///root/unitree_rl_gym/resources/robots/g1_description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
- link right_wrist_pitch_link: geometry collision mesh filename=file:///root/unitree_rl_gym/resources/robots/g1_description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; visual mesh filename=file:///root/unitree_rl_gym/resources/robots/g1_description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
- link right_wrist_roll_link: geometry collision mesh filename=file:///root/unitree_rl_gym/resources/robots/g1_description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; visual mesh filename=file:///root/unitree_rl_gym/resources/robots/g1_description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
- link right_wrist_yaw_link: geometry collision mesh filename=file:///root/unitree_rl_gym/resources/robots/g1_description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; visual mesh filename=file:///root/unitree_rl_gym/resources/robots/g1_description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
- link torso_link: geometry collision mesh filename=file:///root/unitree_rl_gym/resources/robots/g1_description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; visual mesh filename=file:///root/unitree_rl_gym/resources/robots/g1_description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
- link waist_roll_link: geometry visual mesh filename=file:///root/unitree_rl_gym/resources/robots/g1_description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
- link waist_yaw_link: geometry visual mesh filename=file:///root/unitree_rl_gym/resources/robots/g1_description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
- link welder: geometry collision mesh filename=file:///root/unitree_rl_gym/resources/robots/g1_description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; visual mesh filename=file:///root/unitree_rl_gym/resources/robots/g1_description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
