Commit message: 0426

File: resources/robots/g1_description/g1_29dof_rev_1_0_ver4.urdf (robot description, URDF)
Before this commit: robot g1_29dof_rev_1_0, 42 links, 41 joints
Links:
- link left_rubber_hand: geometry collision box size=0.12 0.03 0.08; visual mesh filename=file:///root/unitree_rl_gym/resources/robots/g1_description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

Commit message: update

File: resources/robots/g1_description/g1_29dof_rev_1_0_ver4.urdf (robot description, URDF)
Before this commit: robot g1_29dof_rev_1_0, 42 links, 41 joints
Links:
- link welder: mass 0.3 -> 0.68
