Commit message: working anyway

File: resources/robots/g1_description/g1_29dof_rev_1_0.urdf (robot description, URDF)
Before this commit: robot g1_29dof_rev_1_0, 39 links, 38 joints
Links:
- link left_ankle_roll_link: geometry collision sphere radius=0.005; collision sphere radius=0.005
- link left_rubber_hand: geometry visual mesh filename=meshes/left_rubber_hand.STL
- link pelvis: mass 3.813 -> None
- link right_ankle_roll_link: geometry collision sphere radius=0.005; collision sphere radius=0.005
- link right_rubber_hand: geometry visual mesh filename=meshes/right_rubber_hand.STL
Joints:
- joint left_ankle_pitch_joint: limit lower=-0.87267 upper=0.5236 effort=50 velocity=37 -> lower=-0.87267 upper=0.5236 effort=35 velocity=30
- joint left_ankle_roll_joint: limit lower=-0.2618 upper=0.2618 effort=50 velocity=37 -> lower=-0.2618 upper=0.2618 effort=35 velocity=30
- joint right_ankle_pitch_joint: limit lower=-0.87267 upper=0.5236 effort=50 velocity=37 -> lower=-0.87267 upper=0.5236 effort=35 velocity=30
- joint right_ankle_roll_joint: limit lower=-0.2618 upper=0.2618 effort=50 velocity=37 -> lower=-0.2618 upper=0.2618 effort=35 velocity=30
- joint waist_pitch_joint: limit lower=-0.52 upper=0.52 effort=50 velocity=37 -> lower=-0.52 upper=0.52 effort=35 velocity=30
- joint waist_roll_joint: limit lower=-0.52 upper=0.52 effort=50 velocity=37 -> lower=-0.52 upper=0.52 effort=35 velocity=30
