Commit message: add mid360 link, joint

File: resources/robots/g1_description/g1_29dof_rev_1_0_lidar.urdf (robot description, URDF)
Before this commit: robot g1_29dof_rev_1_0, 42 links, 41 joints
Links:
- removed link end_effector
- removed link welder
- added link left_rubber_hand, mass 0.170; visual mesh filename=meshes/left_rubber_hand.STL
- added link zed2_baro_link
- added link zed2_camera_center; collision mesh filename=meshes/zed2.obj; visual mesh filename=meshes/zed2.obj
- added link zed2_camera_link
- added link zed2_left_camera_frame
- added link zed2_left_camera_optical_frame
- added link zed2_mag_link
- added link zed2_right_camera_frame
- added link zed2_right_camera_optical_frame
- added link zed2_temp_left_link
- added link zed2_temp_right_link
- added link zed_mount; visual mesh filename=meshes/zed_mount.stl
- link head_link: geometry collision mesh filename=meshes/head_link.STL; visual mesh filename=meshes/head_link.STL
- link left_ankle_pitch_link: geometry collision mesh filename=meshes/left_ankle_pitch_link.STL; visual mesh filename=meshes/left_ankle_pitch_link.STL
- link left_ankle_roll_link: geometry collision sphere radius=0.005; collision sphere radius=0.005
- link left_elbow_link: geometry collision mesh filename=meshes/left_elbow_link.STL; visual mesh filename=meshes/left_elbow_link.STL
- link left_hip_pitch_link: geometry collision mesh filename=meshes/left_hip_pitch_link.STL; visual mesh filename=meshes/left_hip_pitch_link.STL
- link left_hip_roll_link: geometry collision mesh filename=meshes/left_hip_roll_link.STL; visual mesh filename=meshes/left_hip_roll_link.STL
- link left_hip_yaw_link: geometry collision mesh filename=meshes/left_hip_yaw_link.STL; visual mesh filename=meshes/left_hip_yaw_link.STL
- link left_knee_link: geometry collision mesh filename=meshes/left_knee_link.STL; visual mesh filename=meshes/left_knee_link.STL
- link left_shoulder_pitch_link: geometry collision cylinder length=0.05 radius=0.03; visual mesh filename=meshes/left_shoulder_pitch_link.STL
- link left_shoulder_roll_link: geometry collision cylinder length=0.03 radius=0.03; visual mesh filename=meshes/left_shoulder_roll_link.STL
- link left_shoulder_yaw_link: geometry collision mesh filename=meshes/left_shoulder_yaw_link.STL; visual mesh filename=meshes/left_shoulder_yaw_link.STL
- link left_wrist_pitch_link: geometry collision mesh filename=meshes/left_wrist_pitch_link.STL; visual mesh filename=meshes/left_wrist_pitch_link.STL
- link left_wrist_roll_link: geometry collision mesh filename=meshes/left_wrist_roll_link.STL; visual mesh filename=meshes/left_wrist_roll_link.STL
- link left_wrist_yaw_link: geometry collision mesh filename=meshes/left_wrist_yaw_link.STL; visual mesh filename=meshes/left_wrist_yaw_link.STL
- link logo_link: geometry collision mesh filename=meshes/logo_link.STL; visual mesh filename=meshes/logo_link.STL
- link pelvis: geometry visual mesh filename=meshes/pelvis.STL
- link pelvis_contour_link: geometry collision mesh filename=meshes/pelvis_contour_link.STL; visual mesh filename=meshes/pelvis_contour_link.STL
- link right_ankle_pitch_link: geometry collision mesh filename=meshes/right_ankle_pitch_link.STL; visual mesh filename=meshes/right_ankle_pitch_link.STL
- link right_ankle_roll_link: geometry collision sphere radius=0.005; collision sphere radius=0.005
- link right_elbow_link: geometry collision mesh filename=meshes/right_elbow_link.STL; visual mesh filename=meshes/right_elbow_link.STL
- link right_hip_pitch_link: geometry collision mesh filename=meshes/right_hip_pitch_link.STL; visual mesh filename=meshes/right_hip_pitch_link.STL
- link right_hip_roll_link: geometry collision mesh filename=meshes/right_hip_roll_link.STL; visual mesh filename=meshes/right_hip_roll_link.STL
- link right_hip_yaw_link: geometry collision mesh filename=meshes/right_hip_yaw_link.STL; visual mesh filename=meshes/right_hip_yaw_link.STL
- link right_knee_link: geometry collision mesh filename=meshes/right_knee_link.STL; visual mesh filename=meshes/right_knee_link.STL
- link right_rubber_hand: geometry visual mesh filename=meshes/right_rubber_hand.STL
- link right_shoulder_pitch_link: geometry collision cylinder length=0.05 radius=0.03; visual mesh filename=meshes/right_shoulder_pitch_link.STL
- link right_shoulder_roll_link: geometry collision cylinder length=0.03 radius=0.03; visual mesh filename=meshes/right_shoulder_roll_link.STL
- link right_shoulder_yaw_link: geometry collision mesh filename=meshes/right_shoulder_yaw_link.STL; visual mesh filename=meshes/right_shoulder_yaw_link.STL
- link right_wrist_pitch_link: geometry collision mesh filename=meshes/right_wrist_pitch_link.STL; visual mesh filename=meshes/right_wrist_pitch_link.STL
- link right_wrist_roll_link: geometry collision mesh filename=meshes/right_wrist_roll_link.STL; visual mesh filename=meshes/right_wrist_roll_link.STL
- link right_wrist_yaw_link: geometry collision mesh filename=meshes/right_wrist_yaw_link.STL; visual mesh filename=meshes/right_wrist_yaw_link.STL
- link torso_link: geometry collision mesh filename=meshes/torso_link_rev_1_0.STL; visual mesh filename=meshes/torso_link_rev_1_0.STL
- link waist_roll_link: geometry visual mesh filename=meshes/waist_roll_link_rev_1_0.STL
- link waist_yaw_link: geometry visual mesh filename=meshes/waist_yaw_link_rev_1_0.STL
Joints:
- removed joint end_effector_joint
- added joint zed2_baro_joint: type fixed, parent zed2_camera_center, child zed2_baro_link, origin xyz=0 0 0 rpy=0 0 0
- added joint zed2_camera_center_joint: type fixed, parent zed2_camera_link, child zed2_camera_center, origin xyz=0 0 0.015 rpy=0 0.05 0
- added joint zed2_left_camera_joint: type fixed, parent zed2_camera_center, child zed2_left_camera_frame, origin xyz=-0.01 0.06 0 rpy=0 0 0
- added joint zed2_left_camera_optical_joint: type fixed, parent zed2_left_camera_frame, child zed2_left_camera_optical_frame, origin xyz=0 0 0 rpy=-1.5707963267948966 0.0 -1.5707963267948966
- added joint zed2_mag_joint: type fixed, parent zed2_camera_center, child zed2_mag_link, origin xyz=0 0 0 rpy=0 0 0
- added joint zed2_right_camera_joint: type fixed, parent zed2_camera_center, child zed2_right_camera_frame, origin xyz=-0.01 -0.06 0 rpy=0 0 0
- added joint zed2_right_camera_optical_joint: type fixed, parent zed2_right_camera_frame, child zed2_right_camera_optical_frame, origin xyz=0 0 0 rpy=-1.5707963267948966 0.0 -1.5707963267948966
- added joint zed2_temp_left_joint: type fixed, parent zed2_left_camera_frame, child zed2_temp_left_link, origin xyz=0 0 0 rpy=0 0 0
- added joint zed2_temp_right_joint: type fixed, parent zed2_right_camera_frame, child zed2_temp_right_link, origin xyz=0 0 0 rpy=0 0 0
- added joint zed_camera_joint: type fixed, parent zed_mount, child zed2_camera_link, origin xyz=0.06920661025 0.0 0.08033553926 rpy=0 0.8234498317 0
- added joint zed_mount_joint: type fixed, parent head_link, child zed_mount, origin xyz=0.0027 0.0 0.3667 rpy=0 -0.04014257279586953 0
- joint left_hand_palm_joint: child welder -> left_rubber_hand

Commit message: adding urdf resources (welder, camera mount, zed, etc.)

File: resources/robots/g1_description/g1_29dof_rev_1_0_lidar.urdf (robot description, URDF)
Before this commit: robot g1_29dof_rev_1_0, 52 links, 51 joints
Links:
- link head_link: geometry collision mesh filename=file:///root/unitree_rl_gym/resources/robots/g1_description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; visual mesh filename=file:///root/unitree_rl_gym/resources/robots/g1_description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
- link left_ankle_pitch_link: geometry collision mesh filename=file:///root/unitree_rl_gym/resources/robots/g1_description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; visual mesh filename=file:///root/unitree_rl_gym/resources/robots/g1_description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
- link left_ankle_roll_link: geometry collision sphere radius=0.005; collision sphere radius=0.005
- link left_elbow_link: geometry collision mesh filename=file:///root/unitree_rl_gym/resources/robots/g1_description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; visual mesh filename=file:///root/unitree_rl_gym/resources/robots/g1_description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
- link left_hip_pitch_link: geometry collision mesh filename=file:///root/unitree_rl_gym/resources/robots/g1_description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; visual mesh filename=file:///root/unitree_rl_gym/resources/robots/g1_description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
- link left_hip_roll_link: geometry collision mesh filename=file:///root/unitree_rl_gym/resources/robots/g1_description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; visual mesh filename=file:///root/unitree_rl_gym/resources/robots/g1_description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
- link left_hip_yaw_link: geometry collision mesh filename=file:///root/unitree_rl_gym/resources/robots/g1_description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; visual mesh filename=file:///root/unitree_rl_gym/resources/robots/g1_description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
- link left_knee_link: geometry collision mesh filename=file:///root/unitree_rl_gym/resources/robots/g1_description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; visual mesh filename=file:///root/unitree_rl_gym/resources/robots/g1_description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
- link left_rubber_hand: geometry visual mesh filename=file:///root/unitree_rl_gym/resources/robots/g1_description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
- link left_shoulder_pitch_link: geometry collision cylinder length=0.05 radius=0.03; visual mesh filename=file:///root/unitree_rl_gym/resources/robots/g1_description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
- link left_shoulder_roll_link: geometry collision cylinder length=0.03 radius=0.03; visual mesh filename=file:///root/unitree_rl_gym/resources/robots/g1_description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
- link left_shoulder_yaw_link: geometry collision mesh filename=file:///root/unitree_rl_gym/resources/robots/g1_description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; visual mesh filename=file:///root/unitree_rl_gym/resources/robots/g1_description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
- link left_wrist_pitch_link: geometry collision mesh filename=file:///root/unitree_rl_gym/resources/robots/g1_description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; visual mesh filename=file:///root/unitree_rl_gym/resources/robots/g1_description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
- link left_wrist_roll_link: geometry collision mesh filename=file:///root/unitree_rl_gym/resources/robots/g1_description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; visual mesh filename=file:///root/unitree_rl_gym/resources/robots/g1_description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
- link left_wrist_yaw_link: geometry collision mesh filename=file:///root/unitree_rl_gym/resources/robots/g1_description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; visual mesh filename=file:///root/unitree_rl_gym/resources/robots/g1_description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
- link logo_link: geometry collision mesh filename=file:///root/unitree_rl_gym/resources/robots/g1_description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; visual mesh filename=file:///root/unitree_rl_gym/resources/robots/g1_description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
- link pelvis: geometry visual mesh filename=file:///root/unitree_rl_gym/resources/robots/g1_description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
- link pelvis_contour_link: geometry collision mesh filename=file:///root/unitree_rl_gym/resources/robots/g1_description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; visual mesh filename=file:///root/unitree_rl_gym/resources/robots/g1_description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
- link right_ankle_pitch_link: geometry collision mesh filename=file:///root/unitree_rl_gym/resources/robots/g1_description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; visual mesh filename=file:///root/unitree_rl_gym/resources/robots/g1_description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
- link right_ankle_roll_link: geometry collision sphere radius=0.005; collision sphere radius=0.005
- link right_elbow_link: geometry collision mesh filename=file:///root/unitree_rl_gym/resources/robots/g1_description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; visual mesh filename=file:///root/unitree_rl_gym/resources/robots/g1_description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
- link right_hip_pitch_link: geometry collision mesh filename=file:///root/unitree_rl_gym/resources/robots/g1_description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; visual mesh filename=file:///root/unitree_rl_gym/resources/robots/g1_description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
- link right_hip_roll_link: geometry collision mesh filename=file:///root/unitree_rl_gym/resources/robots/g1_description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; visual mesh filename=file:///root/unitree_rl_gym/resources/robots/g1_description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
- link right_hip_yaw_link: geometry collision mesh filename=file:///root/unitree_rl_gym/resources/robots/g1_description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; visual mesh filename=file:///root/unitree_rl_gym/resources/robots/g1_description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
- link right_knee_link: geometry collision mesh filename=file:///root/unitree_rl_gym/resources/robots/g1_description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; visual mesh filename=file:///root/unitree_rl_gym/resources/robots/g1_description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
- link right_rubber_hand: geometry visual mesh filename=file:///root/unitree_rl_gym/resources/robots/g1_description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
- link right_shoulder_pitch_link: geometry collision cylinder length=0.05 radius=0.03; visual mesh filename=file:///root/unitree_rl_gym/resources/robots/g1_description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
- link right_shoulder_roll_link: geometry collision cylinder length=0.03 radius=0.03; visual mesh filename=file:///root/unitree_rl_gym/resources/robots/g1_description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
- link right_shoulder_yaw_link: geometry collision mesh filename=file:///root/unitree_rl_gym/resources/robots/g1_description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; visual mesh filename=file:///root/unitree_rl_gym/resources/robots/g1_description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
- link right_wrist_pitch_link: geometry collision mesh filename=file:///root/unitree_rl_gym/resources/robots/g1_description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; visual mesh filename=file:///root/unitree_rl_gym/resources/robots/g1_description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
- link right_wrist_roll_link: geometry collision mesh filename=file:///root/unitree_rl_gym/resources/robots/g1_description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; visual mesh filename=file:///root/unitree_rl_gym/resources/robots/g1_description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
- link right_wrist_yaw_link: geometry collision mesh filename=file:///root/unitree_rl_gym/resources/robots/g1_description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; visual mesh filename=file:///root/unitree_rl_gym/resources/robots/g1_description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
- link torso_link: geometry collision mesh filename=file:///root/unitree_rl_gym/resources/robots/g1_description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; visual mesh filename=file:///root/unitree_rl_gym/resources/robots/g1_description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
- link waist_roll_link: geometry visual mesh filename=file:///root/unitree_rl_gym/resources/robots/g1_description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
- link waist_yaw_link: geometry visual mesh filename=file:///root/unitree_rl_gym/resources/robots/g1_description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
- link zed2_camera_center: geometry collision mesh filename=file:///root/unitree_rl_gym/resources/robots/g1_description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; visual mesh filename=file:///root/unitree_rl_gym/resources/robots/g1_description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
- link zed_mount: geometry visual mesh filename=file:///root/unitree_rl_gym/resources/robots/g1_description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
