Commit message: adding urdf resources (welder, camera mount, zed, etc.)

File: resources/robots/g1_description/g1_29dof_rev_1_0_ver4_camera_mount_v4.urdf (robot description, URDF)
Before this commit: robot g1_29dof_rev_1_0, 52 links, 51 joints
Links:
- removed link right_rubber_hand
- removed link zed2_baro_link
- removed link zed2_camera_center
- removed link zed2_camera_link
- removed link zed2_left_camera_frame
- removed link zed2_left_camera_optical_frame
- removed link zed2_mag_link
- removed link zed2_right_camera_frame
- removed link zed2_right_camera_optical_frame
- removed link zed2_temp_left_link
- removed link zed2_temp_right_link
- removed link zed_mount
- added link camera_color_optical_frame
- added link camera_link
- added link d435_mount_1_link; collision mesh filename=file:///root/unitree_rl_gym/resources/robots/g1_description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 scale=0.001 0.001 0.001; visual mesh filename=file:///root/unitree_rl_gym/resources/robots/g1_description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 scale=0.001 0.001 0.001
- added link d435_mount_2_link; collision mesh filename=file:///root/unitree_rl_gym/resources/robots/g1_description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 scale=0.001 0.001 0.001; visual mesh filename=file:///root/unitree_rl_gym/resources/robots/g1_description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
- added link end_effector; visual sphere radius=0.004
- added link left_sole_link
- added link right_sole_link
- added link welder, mass 0.68; collision mesh filename=file:///root/unitree_rl_gym/resources/robots/g1_description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; visual mesh filename=file:///root/unitree_rl_gym/resources/robots/g1_description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
- added link welder2; collision mesh filename=file:///root/unitree_rl_gym/resources/robots/g1_description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; visual mesh filename=file:///root/unitree_rl_gym/resources/robots/g1_description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
- link d435_link: geometry collision mesh filename=file:///root/unitree_rl_gym/resources/robots/g1_description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; visual mesh filename=file:///root/unitree_rl_gym/resources/robots/g1_description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
- link left_ankle_roll_link: geometry collision box size=0.20820672 0.07558269 0.02; visual mesh filename=file:///root/unitree_rl_gym/resources/robots/g1_description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
- link left_rubber_hand: geometry collision box size=0.12 0.03 0.08; visual mesh filename=file:///root/unitree_rl_gym/resources/robots/g1_description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
- link right_ankle_roll_link: geometry collision box size=0.20820672 0.07558269 0.02; visual mesh filename=file:///root/unitree_rl_gym/resources/robots/g1_description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
Joints:
- removed joint zed2_baro_joint
- removed joint zed2_camera_center_joint
- removed joint zed2_left_camera_joint
- removed joint zed2_left_camera_optical_joint
- removed joint zed2_mag_joint
- removed joint zed2_right_camera_joint
- removed joint zed2_right_camera_optical_joint
- removed joint zed2_temp_left_joint
- removed joint zed2_temp_right_joint
- removed joint zed_camera_joint
- removed joint zed_mount_joint
- added joint camera_color_optical_joint: type fixed, parent camera_link, child camera_color_optical_frame, origin xyz=0 0.015 0 rpy=-1.5707963267948966 0 -1.5707963267948966
- added joint camera_joint: type fixed, parent d435_link, child camera_link, origin xyz=0.018 0 -0.004 rpy=0 -1.5707963267948966 -1.5707963267948966
- added joint d435_mount_1_2: type fixed, parent d435_mount_1_link, child d435_mount_2_link, origin xyz=0 0 0 rpy=0 0 0
- added joint end_effector_joint: type fixed, parent welder, child end_effector, origin xyz=0.0985 0 0.176675 rpy=0 -0.603712724 0
- added joint head_d435_mount_1: type fixed, parent head_link, child d435_mount_1_link, origin xyz=0.012078 0 0.367040 rpy=0 0 3.14159
- added joint left_sole_joint: type fixed, parent left_ankle_roll_link, child left_sole_link, origin xyz=0 0 -0.035 rpy=0 0 0
- added joint right_sole_joint: type fixed, parent right_ankle_roll_link, child right_sole_link, origin xyz=0 0 -0.035 rpy=0 0 0
- added joint welder2_joint: type fixed, parent welder, child welder2, origin xyz=0 0 0 rpy=0 0 0
- joint d435_joint: origin xyz=0.0576235 0.01753 0.42987 rpy=0 0.8307767239493009 0 -> xyz=0.10819156 -0.01456595 0.4446821 rpy=1.8341307 0.1491638 0.805189; parent torso_link -> head_link
- joint right_hand_palm_joint: child right_rubber_hand -> welder

File: resources/robots/g1_description/g1_29dof_rev_1_0_zed2i_with_welder.urdf (robot description, URDF)
Before this commit: robot g1_29dof_rev_1_0, 52 links, 51 joints
Links:
- removed link d435_link
- removed link right_rubber_hand
- removed link zed2_baro_link
- removed link zed2_camera_center
- removed link zed2_camera_link
- removed link zed2_left_camera_frame
- removed link zed2_left_camera_optical_frame
- removed link zed2_mag_link
- removed link zed2_right_camera_frame
- removed link zed2_right_camera_optical_frame
- removed link zed2_temp_left_link
- removed link zed2_temp_right_link
- removed link zed_mount
- added link end_effector; visual sphere radius=0.004
- added link left_sole_link
- added link mount_link, mass 0.25; collision mesh filename=file:///root/unitree_rl_gym/resources/robots/g1_description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 scale=0.001 0.001 0.001; visual mesh filename=file:///root/unitree_rl_gym/resources/robots/g1_description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 scale=0.001 0.001 0.001
- added link right_sole_link
- added link welder, mass 0.68; collision mesh filename=file:///root/unitree_rl_gym/resources/robots/g1_description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; visual mesh filename=file:///root/unitree_rl_gym/resources/robots/g1_description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
- added link welder2; collision mesh filename=file:///root/unitree_rl_gym/resources/robots/g1_description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; visual mesh filename=file:///root/unitree_rl_gym/resources/robots/g1_description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
- added link zed2i_base_link
- added link zed2i_camera_center
- added link zed2i_left_camera_frame
- added link zed2i_left_camera_optical_frame
- added link zed2i_right_camera_frame
- added link zed2i_right_camera_optical_frame
- link left_ankle_roll_link: geometry collision box size=0.20820672 0.07558269 0.02; visual mesh filename=file:///root/unitree_rl_gym/resources/robots/g1_description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
- link left_rubber_hand: geometry collision box size=0.12 0.03 0.08; visual mesh filename=file:///root/unitree_rl_gym/resources/robots/g1_description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
- link right_ankle_roll_link: geometry collision box size=0.20820672 0.07558269 0.02; visual mesh filename=file:///root/unitree_rl_gym/resources/robots/g1_description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
Joints:
- removed joint d435_joint
- removed joint zed2_baro_joint
- removed joint zed2_camera_center_joint
- removed joint zed2_left_camera_joint
- removed joint zed2_left_camera_optical_joint
- removed joint zed2_mag_joint
- removed joint zed2_right_camera_joint
- removed joint zed2_right_camera_optical_joint
- removed joint zed2_temp_left_joint
- removed joint zed2_temp_right_joint
- removed joint zed_camera_joint
- removed joint zed_mount_joint
- added joint end_effector_joint: type fixed, parent welder, child end_effector, origin xyz=0.0985 0 0.176675 rpy=0 -0.603712724 0
- added joint head_to_mount_joint: type fixed, parent head_link, child mount_link, origin xyz=0.11 -0.16 0.352 rpy=0 0 1.0466 
- added joint left_sole_joint: type fixed, parent left_ankle_roll_link, child left_sole_link, origin xyz=0 0 -0.035 rpy=0 0 0
- added joint mount_to_zed2i_joint: type fixed, parent mount_link, child zed2i_base_link, origin xyz=0.116 0.09 0.01 rpy=0 0 -1.5708
- added joint right_sole_joint: type fixed, parent right_ankle_roll_link, child right_sole_link, origin xyz=0 0 -0.035 rpy=0 0 0
- added joint welder2_joint: type fixed, parent welder, child welder2, origin xyz=0 0 0 rpy=0 0 0
- added joint zed2i_camera_center_joint: type fixed, parent zed2i_base_link, child zed2i_camera_center, origin xyz=0 0 0.015 rpy=0 0 0
- added joint zed2i_left_camera_joint: type fixed, parent zed2i_camera_center, child zed2i_left_camera_frame, origin xyz=0 0.06 0 rpy=0 0 0
- added joint zed2i_left_camera_optical_joint: type fixed, parent zed2i_left_camera_frame, child zed2i_left_camera_optical_frame, origin xyz=-0.01 0 0 rpy=-1.5707963267948966 0 -1.5707963267948966
- added joint zed2i_right_camera_joint: type fixed, parent zed2i_camera_center, child zed2i_right_camera_frame, origin xyz=0 -0.06 0 rpy=0 0 0
- added joint zed2i_right_camera_optical_joint: type fixed, parent zed2i_right_camera_frame, child zed2i_right_camera_optical_frame, origin xyz=-0.01 0 0 rpy=-1.5707963267948966 0 -1.5707963267948966
- joint right_hand_palm_joint: child right_rubber_hand -> welder

File: resources/robots/g1_description/g1_29dof_rev_1_0_zed2i_with_welder_v2.urdf (robot description, URDF)
Before this commit: robot g1_29dof_rev_1_0, 52 links, 51 joints
Links:
- removed link d435_link
- removed link right_rubber_hand
- removed link zed2_baro_link
- removed link zed2_camera_center
- removed link zed2_camera_link
- removed link zed2_left_camera_frame
- removed link zed2_left_camera_optical_frame
- removed link zed2_mag_link
- removed link zed2_right_camera_frame
- removed link zed2_right_camera_optical_frame
- removed link zed2_temp_left_link
- removed link zed2_temp_right_link
- removed link zed_mount
- added link end_effector; visual sphere radius=0.004
- added link left_sole_link
- added link mount_link, mass 0.25; collision mesh filename=file:///root/unitree_rl_gym/resources/robots/g1_description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 scale=0.001 0.001 0.001; visual mesh filename=file:///root/unitree_rl_gym/resources/robots/g1_description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 scale=0.001 0.001 0.001
- added link right_sole_link
- added link welder, mass 0.68; collision mesh filename=file:///root/unitree_rl_gym/resources/robots/g1_description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; visual mesh filename=file:///root/unitree_rl_gym/resources/robots/g1_description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
- added link welder2; collision mesh filename=file:///root/unitree_rl_gym/resources/robots/g1_description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; visual mesh filename=file:///root/unitree_rl_gym/resources/robots/g1_description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
- added link zed2i_base_link; visual sphere radius=0.004
- added link zed2i_camera_center; visual sphere radius=0.004
- added link zed2i_left_camera_frame; visual sphere radius=0.004
- added link zed2i_left_camera_optical_frame; visual sphere radius=0.004
- added link zed2i_right_camera_frame
- added link zed2i_right_camera_optical_frame
- link left_ankle_roll_link: geometry collision box size=0.20820672 0.07558269 0.02; visual mesh filename=file:///root/unitree_rl_gym/resources/robots/g1_description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
- link left_rubber_hand: geometry collision box size=0.12 0.03 0.08; visual mesh filename=file:///root/unitree_rl_gym/resources/robots/g1_description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
- link right_ankle_roll_link: geometry collision box size=0.20820672 0.07558269 0.02; visual mesh filename=file:///root/unitree_rl_gym/resources/robots/g1_description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
Joints:
- removed joint d435_joint
- removed joint zed2_baro_joint
- removed joint zed2_camera_center_joint
- removed joint zed2_left_camera_joint
- removed joint zed2_left_camera_optical_joint
- removed joint zed2_mag_joint
- removed joint zed2_right_camera_joint
- removed joint zed2_right_camera_optical_joint
- removed joint zed2_temp_left_joint
- removed joint zed2_temp_right_joint
- removed joint zed_camera_joint
- removed joint zed_mount_joint
- added joint end_effector_joint: type fixed, parent welder, child end_effector, origin xyz=0.0985 0 0.176675 rpy=0 -0.603712724 0
- added joint head_to_mount_joint: type fixed, parent head_link, child mount_link, origin xyz=0.008 0 0.323 rpy=0 0 0 
- added joint left_sole_joint: type fixed, parent left_ankle_roll_link, child left_sole_link, origin xyz=0 0 -0.035 rpy=0 0 0
- added joint mount_to_zed2i_joint: type fixed, parent mount_link, child zed2i_base_link, origin xyz=0.112 -0.01651 0.031 rpy=0 0.349 -0.872
- added joint right_sole_joint: type fixed, parent right_ankle_roll_link, child right_sole_link, origin xyz=0 0 -0.035 rpy=0 0 0
- added joint welder2_joint: type fixed, parent welder, child welder2, origin xyz=0 0 0 rpy=0 0 0
- added joint zed2i_camera_center_joint: type fixed, parent zed2i_base_link, child zed2i_camera_center, origin xyz=0 0 0.015 rpy=0 0 0
- added joint zed2i_left_camera_joint: type fixed, parent zed2i_camera_center, child zed2i_left_camera_frame, origin xyz=0 0.06 0 rpy=0 0 0
- added joint zed2i_left_camera_optical_joint: type fixed, parent zed2i_left_camera_frame, child zed2i_left_camera_optical_frame, origin xyz=-0.01 0 0 rpy=-1.5707963267948966 0 -1.5707963267948966
- added joint zed2i_right_camera_joint: type fixed, parent zed2i_camera_center, child zed2i_right_camera_frame, origin xyz=0 -0.06 0 rpy=0 0 0
- added joint zed2i_right_camera_optical_joint: type fixed, parent zed2i_right_camera_frame, child zed2i_right_camera_optical_frame, origin xyz=-0.01 0 0 rpy=-1.5707963267948966 0 -1.5707963267948966
- joint right_hand_palm_joint: child right_rubber_hand -> welder

File: resources/robots/g1_description/g1_29dof_rev_1_0_zed_with_welder.urdf (robot description, URDF)
Before this commit: robot g1_29dof_rev_1_0, 52 links, 51 joints
Links:
- removed link d435_link
- removed link right_rubber_hand
- removed link zed_mount
- added link end_effector; visual sphere radius=0.004
- added link left_sole_link
- added link mount_link, mass 0.25; collision mesh filename=file:///root/unitree_rl_gym/resources/robots/g1_description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 scale=0.001 0.001 0.001; visual mesh filename=file:///root/unitree_rl_gym/resources/robots/g1_description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 scale=0.001 0.001 0.001
- added link right_sole_link
- added link welder, mass 0.68; collision mesh filename=file:///root/unitree_rl_gym/resources/robots/g1_description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; visual mesh filename=file:///root/unitree_rl_gym/resources/robots/g1_description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
- added link welder2; collision mesh filename=file:///root/unitree_rl_gym/resources/robots/g1_description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; visual mesh filename=file:///root/unitree_rl_gym/resources/robots/g1_description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
- link left_ankle_roll_link: geometry collision box size=0.20820672 0.07558269 0.02; visual mesh filename=file:///root/unitree_rl_gym/resources/robots/g1_description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
- link left_rubber_hand: geometry collision box size=0.12 0.03 0.08; visual mesh filename=file:///root/unitree_rl_gym/resources/robots/g1_description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
- link right_ankle_roll_link: geometry collision box size=0.20820672 0.07558269 0.02; visual mesh filename=file:///root/unitree_rl_gym/resources/robots/g1_description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
- link zed2_camera_center: mass None -> 0.17; geometry collision mesh filename=file:///root/unitree_rl_gym/resources/robots/g1_description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 scale=0.001 0.001 0.001; visual mesh filename=file:///root/unitree_rl_gym/resources/robots/g1_description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 scale=0.001 0.001 0.001
Joints:
- removed joint d435_joint
- removed joint zed_camera_joint
- removed joint zed_mount_joint
- added joint end_effector_joint: type fixed, parent welder, child end_effector, origin xyz=0.0985 0 0.176675 rpy=0 -0.603712724 0
- added joint head_to_mount_joint: type fixed, parent head_link, child mount_link, origin xyz=0.11 -0.16 0.352 rpy=0 0 1.0466 
- added joint left_sole_joint: type fixed, parent left_ankle_roll_link, child left_sole_link, origin xyz=0 0 -0.035 rpy=0 0 0
- added joint mount_to_zed2i_joint: type fixed, parent mount_link, child zed2_camera_link, origin xyz=0 -0.002 -0.022 rpy=0 0 0
- added joint right_sole_joint: type fixed, parent right_ankle_roll_link, child right_sole_link, origin xyz=0 0 -0.035 rpy=0 0 0
- added joint welder2_joint: type fixed, parent welder, child welder2, origin xyz=0 0 0 rpy=0 0 0
- joint right_hand_palm_joint: child right_rubber_hand -> welder
- joint zed2_camera_center_joint: origin xyz=0 0 0.015 rpy=0 0.05 0 -> xyz=0 0 0 rpy=0 0 0
