Commit message: 1013 saved

File: resources/robots/g1_description/g1_29dof_rev_1_0_zed2i_with_welder_v2.urdf (robot description, URDF)
Before this commit: robot g1_29dof_rev_1_0, 51 links, 50 joints
Joints:
- joint zed2i_left_camera_optical_joint: origin xyz=-0.01 0 0 rpy=-1.5707963267948966 0 -1.5707963267948966 -> xyz=-0.00668378 0.01467285 0.03236308 rpy=-1.5707963267948966 0 -1.5707963267948966
