Commit message: correct d435 location

File: resources/robots/g1_description/g1_29dof_rev_1_0_d435_with_welder_v2.urdf (robot description, URDF)
Before this commit: robot g1_29dof_rev_1_0, 52 links, 50 joints
Joints:
- added joint camera_link_joint: type fixed, parent torso_link, child camera_link, origin xyz=0.0576235 0.01753 0.42987 rpy=0 0.8307767239493009 0
