Commit message: removing welder from d435 urdf and renaming it

File: resources/robots/g1_description/g1_29dof_rev_1_0_d435.urdf (robot description, URDF)
Before this commit: robot g1_29dof_rev_1_0, 52 links, 51 joints
Links:
- removed link welder
Joints:
- removed joint right_hand_palm_joint
- joint end_effector_joint: origin xyz=0.0 0 0.0 rpy=0 0 0 -> xyz=0.0455 0.003 0 rpy=0 0 0; parent welder -> right_wrist_yaw_link

Commit message: updates to testing hand delta

File: resources/robots/g1_description/g1_29dof_rev_1_0_d435.urdf (robot description, URDF)
Before this commit: robot g1_29dof_rev_1_0, 51 links, 50 joints
Joints:
- joint end_effector_joint: parent right_wrist_yaw_link -> left_wrist_yaw_link
