Commit message: update

File: resources/robots/g1_description/g1_29dof_rev_1_0_zed2i_with_welder_v3.urdf (robot description, URDF)
Before this commit: robot g1_29dof_rev_1_0, 50 links, 49 joints
Links:
- added link tag_10; visual sphere radius=0.004
- added link tag_11; visual sphere radius=0.004
- added link tag_12; visual sphere radius=0.004
Joints:
- added joint tag_10_joint: type fixed, parent welder, child tag_10, origin xyz=0.0385 0.0215 0.041155 rpy=0 1.5707963 1.5707963
- added joint tag_11_joint: type fixed, parent welder, child tag_11, origin xyz=0.0385 0.0215 0.001155 rpy=0 1.5707963 1.5707963
- added joint tag_12_joint: type fixed, parent welder, child tag_12, origin xyz=0.0385 0.0215 -0.038845 rpy=0 1.5707963 1.5707963
- joint zed2i_left_camera_optical_joint: origin xyz=-0.01 0 0 rpy=-1.5707963267948966 0 -1.5707963267948966 -> xyz=0.01395555 -0.00256978 -0.00997866 rpy=-1.63664046 -0.00976016 -1.6094062

Commit message: 0920 MD success

File: resources/robots/g1_description/g1_29dof_rev_1_0_zed2i_with_welder_v3.urdf (robot description, URDF)
Before this commit: robot g1_29dof_rev_1_0, 53 links, 52 joints
Joints:
- joint zed2i_left_camera_optical_joint: origin xyz=0.01395555 -0.00256978 -0.00997866 rpy=-1.63664046 -0.00976016 -1.6094062 -> xyz=0.00314297  0.00466147 -0.00981058 rpy=-1.54015865 -0.01350367 -1.56338791

Commit message: 0921 welding success

File: resources/robots/g1_description/g1_29dof_rev_1_0_zed2i_with_welder_v3.urdf (robot description, URDF)
Before this commit: robot g1_29dof_rev_1_0, 53 links, 52 joints
Joints:
- joint zed2i_left_camera_optical_joint: origin xyz=0.00314297  0.00466147 -0.00981058 rpy=-1.54015865 -0.01350367 -1.56338791 -> xyz=0.00330548  0.00459355 -0.00980306 rpy=-1.54007246 -0.01351019 -1.56349733

Commit message: update

File: resources/robots/g1_description/g1_29dof_rev_1_0_zed2i_with_welder_v3.urdf (robot description, URDF)
Before this commit: robot g1_29dof_rev_1_0, 53 links, 52 joints
Joints:
- joint zed2i_left_camera_optical_joint: origin xyz=0.00330548  0.00459355 -0.00980306 rpy=-1.54007246 -0.01351019 -1.56349733 -> xyz=0.00342784  0.00457491 -0.00980677 rpy=-1.54007993 -0.01349432 -1.56356784

Commit message: rooftop 1002

File: resources/robots/g1_description/g1_29dof_rev_1_0_zed2i_with_welder_v3.urdf (robot description, URDF)
Before this commit: robot g1_29dof_rev_1_0, 53 links, 52 joints
Joints:
- joint zed2i_left_camera_optical_joint: origin xyz=0.00342784  0.00457491 -0.00980677 rpy=-1.54007993 -0.01349432 -1.56356784 -> xyz=0.00350179  0.00458972 -0.00981216 rpy=-1.54009763 -0.01348875 -1.56361833

Commit message: demo

File: resources/robots/g1_description/g1_29dof_rev_1_0_zed2i_with_welder_v3.urdf (robot description, URDF)
Before this commit: robot g1_29dof_rev_1_0, 53 links, 52 joints
Links:
- link welder: mass 0.68 -> 0.3
Joints:
- joint zed2i_left_camera_optical_joint: origin xyz=0.00350179  0.00458972 -0.00981216 rpy=-1.54009763 -0.01348875 -1.56361833 -> xyz=0.00360727  0.00401995 -0.01006136 rpy=-1.54069048 -0.01339886 -1.56305672
